File: Ladder LEDs v1/Ladder LEDs v1.kicad_pcb (KiCad board)
At the start: 2 copper layers, 37.8 x 33.7 mm, 16 parts, among them J1 01×03 Molex Nanofit Header, J2 02×02 Molex Nanofit Header, J3 Conn_01x04_Pin

Commit message: Created Gerber files for OSH Park
Connections:
- J2 pad 1: Net-(J2-DATA) -> Net-(J1-5V)
- J2 pad 2: Net-(J1-5V) -> Net-(J2-DATA)
Routing:
- net GND: track 2.43 -> 5.91 mm, vias 1 -> 2
- net Net-(J2-DATA): track 14.6 -> 16.1 mm
