File: Ladder LEDs/Ladder LEDs.kicad_pcb (KiCad board)
At the start: 2 copper layers, 37.8 x 33.7 mm, 16 parts, among them J1 01×03 Molex Nanofit Header, J2 02×02 Molex Nanofit Header, J3 Conn_01x04_Pin

Commit message: Trimmed BOM, added 3D models
Changed lines of the file:
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@@
     (pad "4" thru_hole circle (at 0 0 334.5) (size 2.5 2.5) (drill 1.57) (layers "*.Cu" "*.Mask")
       (net 8 "unconnected-(J3-Pin_4-Pad4)") (pinfunction "Pin_4") (pintype "passive+no_connect"))
+    (model "${KICAD6_3DMODEL_DIR}/Custom/Ladder-LEDs-3D-Models/keystone-PN7779.STEP"
+      (offset (xyz 2.5 -5 -3))
+      (scale (xyz 1 1 1))
+      (rotate (xyz 90 0 180))
+    )
   )
   (footprint "LadderLEDLib:Molex 105405-1104" (layer "F.Cu")
@@
     (pad "6" smd rect (at 7.04 0 180) (size 1.1 8.2) (layers "F.Cu" "F.Paste" "F.Mask")
       (thermal_bridge_angle 45))
+    (model "${KICAD6_3DMODEL_DIR}/Custom/Ladder-LEDs-3D-Models/1054051104.stp"
+      (offset (xyz 3.8 4.5 3.25))
+      (scale (xyz 1 1 1))
+      (rotate (xyz -90 0 0))
+    )
   )
   (footprint "LadderLEDLib:Molex 1054302103" (layer "F.Cu")
@@
     (pad "5" smd rect (at 9.54 0 334) (size 1.1 8.2) (layers "F.Cu" "F.Paste" "F.Mask")
       (thermal_bridge_angle 45))
+    (model "${KICAD6_3DMODEL_DIR}/Custom/Ladder-LEDs-3D-Models/1054302103.stp"
+      (offset (xyz 4.75 0 2))
+      (scale (xyz 1 1 1))
+      (rotate (xyz -90 0 0))
+    )
   )
   (footprint "Capacitor_SMD:C_0805_2012Metric_Pad1.18x1.45mm_HandSolder" (layer "B.Cu")
@@
         (effects (font (size 1 1) (thickness 0.15)) (justify mirror))
     )
-    (fp_text value "0.1u" (at 51.591495 -14.318437 27) (layer "B.Fab")
+    (fp_text value "0.1u" (at -5.092684 -4.224889 27) (layer "B.Fab")
         (effects (font (size 1 1) (thickness 0.15)) (justify mirror))
     )
@@
     (pad "4" smd roundrect (at 2.4 1.7 328) (size 1.6 1.2) (layers "B.Cu" "B.Paste" "B.Mask") (roundrect_rratio 0.06561666667)
       (net 11 "Net-(U2-DOUT)") (pinfunction "DIN") (pintype "input") (thermal_bridge_angle 45))
+    (model "${KICAD6_3DMODEL_DIR}/Custom/Ladder-LEDs-3D-Models/IN-PI55QATPRPGPBPW-XX.STEP"
+      (offset (xyz -2.75 -2.5 0))
+      (scale (xyz 1 1 1))
+      (rotate (xyz -90 0 0))
+    )
   )
   (footprint "Capacitor_SMD:C_0805_2012Metric_Pad1.18x1.45mm_HandSolder" (layer "B.Cu")
@@
     (pad "4" smd roundrect (at 2.4 1.7 274) (size 1.6 1.2) (layers "B.Cu" "B.Paste" "B.Mask") (roundrect_rratio 0.06561666667)
       (net 10 "Net-(U1-DOUT)") (pinfunction "DIN") (pintype "input") (thermal_bridge_angle 45))
+    (model "${KICAD6_3DMODEL_DIR}/Custom/Ladder-LEDs-3D-Models/IN-PI55QATPRPGPBPW-XX.STEP"
+      (offset (xyz -2.75 -2.5 0))
+      (scale (xyz 1 1 1))
+      (rotate (xyz -90 0 0))
+    )
   )
   (footprint "Capacitor_SMD:C_0805_2012Metric_Pad1.18x1.45mm_HandSolder" (layer "B.Cu")
@@
     (pad "4" smd roundrect (at 2.4 1.7 239) (size 1.6 1.2) (layers "B.Cu" "B.Paste" "B.Mask") (roundrect_rratio 0.06561666667)
       (net 9 "Net-(U1-DIN)") (pinfunction "DIN") (pintype "input") (thermal_bridge_angle 45))
+    (model "${KICAD6_3DMODEL_DIR}/Custom/Ladder-LEDs-3D-Models/IN-PI55QATPRPGPBPW-XX.STEP"
+      (offset (xyz -2.75 -2.5 0))
+      (scale (xyz 1 1 1))
+      (rotate (xyz -90 0 0))
+    )
   )
   (footprint "LadderLEDLib:IN-PI55QATPRPGPBPW-XX" (layer "B.Cu")
@@
     (pad "4" smd roundrect (at 2.4 1.7 59) (size 1.6 1.2) (layers "B.Cu" "B.Paste" "B.Mask") (roundrect_rratio 0.06561666667)
       (net 13 "Net-(U4-DOUT)") (pinfunction "DIN") (pintype "input") (thermal_bridge_angle 45))
+    (model "${KICAD6_3DMODEL_DIR}/Custom/Ladder-LEDs-3D-Models/IN-PI55QATPRPGPBPW-XX.STEP"
+      (offset (xyz -2.75 -2.5 0))
+      (scale (xyz 1 1 1))
+      (rotate (xyz -90 0 0))
+    )
   )
   (footprint "LadderLEDLib:IN-PI55QATPRPGPBPW-XX" (layer "B.Cu")
@@
     (pad "4" smd roundrect (at 2.4 1.7 154.5) (size 1.6 1.2) (layers "B.Cu" "B.Paste" "B.Mask") (roundrect_rratio 0.06561666667)
       (net 14 "Net-(U5-DOUT)") (pinfunction "DIN") (pintype "input") (thermal_bridge_angle 45))
+    (model "${KICAD6_3DMODEL_DIR}/Custom/Ladder-LEDs-3D-Models/IN-PI55QATPRPGPBPW-XX.STEP"
+      (offset (xyz -2.75 -2.5 0))
+      (scale (xyz 1 1 1))
+      (rotate (xyz -90 0 0))
+    )
   )
   (footprint "Capacitor_SMD:C_0805_2012Metric_Pad1.18x1.45mm_HandSolder" (layer "B.Cu")
@@
     (pad "4" smd roundrect (at 2.4 1.7 27) (size 1.6 1.2) (layers "B.Cu" "B.Paste" "B.Mask") (roundrect_rratio 0.06561666667)
       (net 12 "Net-(U3-DOUT)") (pinfunction "DIN") (pintype "input") (thermal_bridge_angle 45))
+    (model "${KICAD6_3DMODEL_DIR}/Custom/Ladder-LEDs-3D-Models/IN-PI55QATPRPGPBPW-XX.STEP"
+      (offset (xyz -2.75 -2.5 0))
+      (scale (xyz 1 1 1))
+      (rotate (xyz -90 0 0))
+    )
   )
   (footprint "Capacitor_SMD:C_0805_2012Metric_Pad1.18x1.45mm_HandSolder" (layer "B.Cu")
@@
       (xy 159.435613 114.764624)
       (xy 159.435612 114.764624)
-      (xy 159.435612 114.764624)
       (xy 159.435608 114.764626)
