File: Ladder LEDs/Ladder LEDs.kicad_sch (KiCad schematic)
At the start: 16 parts, among them J1 01×03 Molex Nanofit Header, J2 02×02 Molex Nanofit Header, J3 Conn_01x04_Pin

Commit message: Trimmed BOM, added 3D models
Parts:
- J1: MPN (none) -> 1054302103
- J2: MPN (none) -> 1054051104
Other:
- company: (none) -> Cephalophore
- title: (none) -> Ladder-LEDs Single Board
Changed lines of the file:
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@@
 (kicad_sch (version 20230121) (generator eeschema)
   (paper "A4")
+  (title_block
+    (title "Ladder-LEDs Single Board")
+    (rev "1")
+    (company "Cephalophore")
+  )
   (junction (at 132.08 83.82) (diameter 0) (color 0 0 0 0)
   )
@@
     (pin "4")
     (instances
-      (project "Ladder LEDs v1"
+      (project "Ladder LEDs"
         (path "/e491d8ef-51ef-4630-8903-9fd9bed65440"
           (reference "J3") (unit 1)
@@
     (pin "2")
     (instances
-      (project "Ladder LEDs v1"
+      (project "Ladder LEDs"
         (path "/e491d8ef-51ef-4630-8903-9fd9bed65440"
           (reference "C5") (unit 1)
@@
     (pin "4")
     (instances
-      (project "Ladder LEDs v1"
+      (project "Ladder LEDs"
         (path "/e491d8ef-51ef-4630-8903-9fd9bed65440"
           (reference "U2") (unit 1)
@@
     (pin "2")
     (instances
-      (project "Ladder LEDs v1"
+      (project "Ladder LEDs"
         (path "/e491d8ef-51ef-4630-8903-9fd9bed65440"
           (reference "C4") (unit 1)
@@
       (effects (font (size 1.27 1.27)) hide)
     )
-    (property "MPN" "" (at 151.13 179.07 0)
+    (property "MPN" "1054051104" (at 151.13 179.07 0)
       (effects (font (size 1.27 1.27)) hide)
     )
@@
     (pin "4")
     (instances
-      (project "Ladder LEDs v1"
+      (project "Ladder LEDs"
         (path "/e491d8ef-51ef-4630-8903-9fd9bed65440"
           (reference "J2") (unit 1)
@@
     (pin "1")
     (instances
-      (project "Ladder LEDs v1"
+      (project "Ladder LEDs"
         (path "/e491d8ef-51ef-4630-8903-9fd9bed65440"
           (reference "#PWR02") (unit 1)
@@
     (pin "1")
     (instances
-      (project "Ladder LEDs v1"
+      (project "Ladder LEDs"
         (path "/e491d8ef-51ef-4630-8903-9fd9bed65440"
           (reference "#PWR06") (unit 1)
@@
     (pin "2")
     (instances
-      (project "Ladder LEDs v1"
+      (project "Ladder LEDs"
         (path "/e491d8ef-51ef-4630-8903-9fd9bed65440"
           (reference "C2") (unit 1)
@@
     (pin "2")
     (instances
-      (project "Ladder LEDs v1"
+      (project "Ladder LEDs"
         (path "/e491d8ef-51ef-4630-8903-9fd9bed65440"
           (reference "C6") (unit 1)
@@
     (pin "4")
     (instances
-      (project "Ladder LEDs v1"
+      (project "Ladder LEDs"
         (path "/e491d8ef-51ef-4630-8903-9fd9bed65440"
           (reference "U5") (unit 1)
@@
     (pin "1")
     (instances
-      (project "Ladder LEDs v1"
+      (project "Ladder LEDs"
         (path "/e491d8ef-51ef-4630-8903-9fd9bed65440"
           (reference "#PWR07") (unit 1)
@@
     (pin "2")
     (instances
-      (project "Ladder LEDs v1"
+      (project "Ladder LEDs"
         (path "/e491d8ef-51ef-4630-8903-9fd9bed65440"
           (reference "C1") (unit 1)
@@
     (pin "2")
     (instances
-      (project "Ladder LEDs v1"
+      (project "Ladder LEDs"
         (path "/e491d8ef-51ef-4630-8903-9fd9bed65440"
           (reference "R1") (unit 1)
@@
     (pin "4")
     (instances
-      (project "Ladder LEDs v1"
+      (project "Ladder LEDs"
         (path "/e491d8ef-51ef-4630-8903-9fd9bed65440"
           (reference "U6") (unit 1)
@@
     (pin "4")
     (instances
-      (project "Ladder LEDs v1"
+      (project "Ladder LEDs"
         (path "/e491d8ef-51ef-4630-8903-9fd9bed65440"
           (reference "U4") (unit 1)
@@
     (pin "1")
     (instances
-      (project "Ladder LEDs v1"
+      (project "Ladder LEDs"
         (path "/e491d8ef-51ef-4630-8903-9fd9bed65440"
           (reference "#PWR04") (unit 1)
@@
     (pin "1")
     (instances
-      (project "Ladder LEDs v1"
+      (project "Ladder LEDs"
         (path "/e491d8ef-51ef-4630-8903-9fd9bed65440"
           (reference "#PWR03") (unit 1)
@@
     (pin "1")
     (instances
-      (project "Ladder LEDs v1"
+      (project "Ladder LEDs"
         (path "/e491d8ef-51ef-4630-8903-9fd9bed65440"
           (reference "#PWR01") (unit 1)
@@
     (pin "1")
     (instances
-      (project "Ladder LEDs v1"
+      (project "Ladder LEDs"
         (path "/e491d8ef-51ef-4630-8903-9fd9bed65440"
           (reference "#PWR05") (unit 1)
@@
       (effects (font (size 1.27 1.27)) hide)
     )
-    (property "MPN" "" (at 184.15 24.13 0)
+    (property "MPN" "1054302103" (at 184.15 24.13 0)
       (effects (font (size 1.27 1.27)) hide)
     )
@@
     (pin "3")
     (instances
-      (project "Ladder LEDs v1"
+      (project "Ladder LEDs"
         (path "/e491d8ef-51ef-4630-8903-9fd9bed65440"
           (reference "J1") (unit 1)
@@
     (pin "4")
     (instances
-      (project "Ladder LEDs v1"
+      (project "Ladder LEDs"
         (path "/e491d8ef-51ef-4630-8903-9fd9bed65440"
           (reference "U3") (unit 1)
@@
     (pin "2")
     (instances
-      (project "Ladder LEDs v1"
+      (project "Ladder LEDs"
         (path "/e491d8ef-51ef-4630-8903-9fd9bed65440"
           (reference "C3") (unit 1)
@@
     (pin "4")
     (instances
-      (project "Ladder LEDs v1"
+      (project "Ladder LEDs"
         (path "/e491d8ef-51ef-4630-8903-9fd9bed65440"
           (reference "U1") (unit 1)
